Commit message: Add MoveIt service to docker-compose, update controllers and URDF configurations for improved robot control

File: AMR_COBOT_urdf/urdf/AMR_COBOT.urdf (robot description, URDF)
Before this commit: robot AMR_COBOT, 18 links, 17 joints
Joints:
- joint 1_hand_joint: limit lower=-0.025 upper=0 effort=0 velocity=0 -> lower=-0.025 upper=0 effort=50 velocity=0.2
- joint 2_hand_joint: limit lower=0 upper=0.025 effort=0 velocity=0 -> lower=0 upper=0.025 effort=50 velocity=0.2
